File: Board/Board.sch (KiCad schematic (older format))
At the start: 14 parts, among them J1 Bluetooth, J2 Conn_01x04_Female, J3 AudioJack3, J4 Conn_01x03_Female, J5 Conn_01x04_Female, J6 Voltage In 1, J7 Voltage In 2, J8 TrnasistorNPN

Commit message: now its perfect
Parts:
- removed A1: Arduino_Nano_v3.x, Module:Arduino_Nano, symbol MCU_Module:Arduino_Nano_v3.x
- removed C1: CAP, Capacitors:CPOL-RADIAL-2.5MM-5MM, symbol pspice:CAP
- removed J1: Bluetooth, Connector_PinHeader_2.54mm:PinHeader_1x06_P2.54mm_Vertical, symbol Connector:Conn_01x06_Female
- removed J3: AudioJack3, Connector_PinHeader_2.54mm:PinHeader_1x03_P2.54mm_Vertical, symbol Connector:AudioJack3
- removed J4: Conn_01x03_Female, Connector_PinHeader_2.54mm:PinHeader_1x03_P2.54mm_Vertical, symbol Connector:Conn_01x03_Female
- removed J8: TrnasistorNPN, Connector_PinHeader_2.54mm:PinHeader_1x03_P2.54mm_Vertical, symbol Connector:Conn_01x03_Female
- removed R1: 2K, Connector_PinHeader_2.54mm:PinHeader_1x02_P2.54mm_Vertical, symbol Device:R
- removed R2: 1K, Connector_PinHeader_2.54mm:PinHeader_1x02_P2.54mm_Vertical, symbol Device:R
- added DRV3: Y1 Driver, DRV8825_STEPPER_MOTOR_DRIVER_CARRIER:IC_DRV8825_STEPPER_MOTOR_DRIVER_CARRIER, symbol Board-rescue:DRV8825_STEPPER_MOTOR_DRIVER_CARRIER-DRV8825_STEPPER_MOTOR_DRIVER_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
- added DRV4: Y2 Driver, DRV8825_STEPPER_MOTOR_DRIVER_CARRIER:IC_DRV8825_STEPPER_MOTOR_DRIVER_CARRIER, symbol Board-rescue:DRV8825_STEPPER_MOTOR_DRIVER_CARRIER-DRV8825_STEPPER_MOTOR_DRIVER_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
- added DRV5: Z1 Driver, DRV8825_STEPPER_MOTOR_DRIVER_CARRIER:IC_DRV8825_STEPPER_MOTOR_DRIVER_CARRIER, symbol Board-rescue:DRV8825_STEPPER_MOTOR_DRIVER_CARRIER-DRV8825_STEPPER_MOTOR_DRIVER_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
- added J1, J3, J4: Conn_01x04_Female, Connector_PinHeader_2.54mm:PinHeader_1x04_P2.54mm_Vertical, symbol Connector:Conn_01x04_Female
- added J10: Conn_01x05_Female, Connector_PinHeader_2.54mm:PinHeader_1x05_P2.54mm_Vertical, symbol Connector:Conn_01x05_Female
- added J11: CAP, Connector_PinHeader_2.54mm:PinHeader_1x02_P2.54mm_Vertical, symbol Connector:Conn_01x02_Female
- added J8: Conn_02x05_Odd_Even, Connector_PinHeader_2.54mm:PinHeader_2x05_P2.54mm_Vertical, symbol Connector_Generic:Conn_02x05_Odd_Even
- added J9: Probe Header, Connector_PinHeader_2.54mm:PinHeader_1x02_P2.54mm_Vertical, symbol Connector:Conn_01x02_Female
- added U1: Teensy4.1, teensy:Teensy41, symbol teensy:Teensy4.1
- DRV1: value DRV8825_STEPPER_MOTOR_DRIVER_CARRIER -> X1 Driver; symbol DRV8825_STEPPER_MOTOR_DRIVER_CARRIER:DRV8825_STEPPER_MOTOR_DRIVER_CARRIER -> Board-rescue:DRV8825_STEPPER_MOTOR_DRIVER_CARRIER-DRV8825_STEPPER_MOTOR_DRIVER_CARRIER
- DRV2: value DRV8825_STEPPER_MOTOR_DRIVER_CARRIER -> X2 Driver; symbol DRV8825_STEPPER_MOTOR_DRIVER_CARRIER:DRV8825_STEPPER_MOTOR_DRIVER_CARRIER -> Board-rescue:DRV8825_STEPPER_MOTOR_DRIVER_CARRIER-DRV8825_STEPPER_MOTOR_DRIVER_CARRIER
Connections:
- net 12V: now also DRV3.16 (VMOT), DRV4.16 (VMOT), DRV5.16 (VMOT), J11.1 (Pin_1)
- net GND: now also DRV3.15 (GND_MOT), DRV3.9 (GND), DRV4.15 (GND_MOT), DRV4.9 (GND), DRV5.15 (GND_MOT), DRV5.9 (GND), J10.1 (Pin_1), J11.2 (Pin_2), J8.1 (Pin_1), J8.3 (Pin_3), J8.5 (Pin_5), J8.7 (Pin_7), J8.9 (Pin_9), J9.2 (Pin_2), U1.1 (GND), U1.47 (GND)
- net STEP2: now reaches DRV2.7 (STEP)
- net STEP2: now also U1.11 (9_OUT1C)
- net 3V: now reaches DRV2.1 (~EN)
- net 3V: now also DRV1.1 (~EN), DRV1.4 (M2), DRV1.5 (~RST), DRV1.6 (~SLP), DRV2.4 (M2), DRV2.5 (~RST), DRV2.6 (~SLP), DRV3.1 (~EN), DRV3.4 (M2), DRV3.5 (~RST), DRV3.6 (~SLP), DRV4.1 (~EN), DRV4.4 (M2), DRV4.5 (~RST), DRV4.6 (~SLP), DRV5.1 (~EN), DRV5.4 (M2), DRV5.5 (~RST), DRV5.6 (~SLP), J10.2 (Pin_2), U1.15 (3V3), U1.46 (3V3)
- net DIR1: now reaches DRV1.8 (DIR)
- net DIR1: now also U1.5 (3_LRCLK2)
- net STEP1: now reaches DRV1.7 (STEP)
- net STEP1: now also U1.4 (2_OUT2)
- net DIR2: now reaches DRV2.8 (DIR)
- net DIR2: now also U1.10 (8_TX2_IN1)
- removed net 5V: DRV1.10 (~FLT), DRV1.2 (M0), DRV1.3 (M1), DRV1.5 (~RST), DRV1.6 (~SLP), DRV2.10 (~FLT), DRV2.2 (M0), DRV2.3 (M1), DRV2.5 (~RST), DRV2.6 (~SLP)
- new net: DRV3.11 (A2), J1.1 (Pin_1)
- new net: DRV3.12 (A1), J1.2 (Pin_2)
- new net: DRV3.13 (B1), J1.3 (Pin_3)
- new net: DRV3.14 (B2), J1.4 (Pin_4)
- new net: DRV5.11 (A2), J4.1 (Pin_1)
- new net: DRV5.12 (A1), J4.2 (Pin_2)
- new net: DRV5.13 (B1), J4.3 (Pin_3)
- new net: DRV5.14 (B2), J4.4 (Pin_4)
- new net: DRV4.11 (A2), J3.1 (Pin_1)
- new net: DRV4.12 (A1), J3.2 (Pin_2)
- new net: DRV4.13 (B1), J3.3 (Pin_3)
- new net: DRV4.14 (B2), J3.4 (Pin_4)
- new net DIR3: DRV3.8 (DIR), U1.6 (4_BCLK2)
- new net DIR4: DRV4.8 (DIR), U1.12 (10_CS_MQSR)
- new net DIR5: DRV5.8 (DIR), U1.8 (6_OUT1D)
- new net Limit1: J8.10 (Pin_10), U1.41 (19_A5_SCL)
- new net Limit2: J8.8 (Pin_8), U1.42 (20_A6_TX5_LRCLK1)
- new net Limit3: J8.6 (Pin_6), U1.43 (21_A7_RX5_BCLK1)
- new net Limit4: J8.4 (Pin_4), U1.44 (22_A8_CTX1)
- new net Limit5: J8.2 (Pin_2), U1.45 (23_A9_CRX1_MCLK1)
- new net PROBE: J9.1 (Pin_1), U1.37 (15_A1_RX3_SPDIF_IN)
- new net STEP3: DRV3.7 (STEP), U1.7 (5_IN2)
- new net STEP4: DRV4.7 (STEP), U1.13 (11_MOSI_CTX1)
- new net STEP5: DRV5.7 (STEP), U1.9 (7_RX2_OUT1A)
- new net SpindleDIR: J10.4 (Pin_4), U1.33 (41_A17)
- new net SpindleEN: J10.5 (Pin_5), U1.32 (40_A16)
- new net SpindlePWM: J10.3 (Pin_3), U1.35 (13_SCK_LED)
- no-connect marks 20 -> 10
Other:
- moved on the sheet: DRV1, DRV2, J2, J5, J6, J7
